File: pcb/nano isp pcb.kicad_pcb (KiCad board)
At the start: 2 copper layers, 72.4 x 20.3 mm, 10 parts, among them J1 Conn_01x03, J2 Conn_01x06, J3 Conn_02x03_Top_Bottom, U1 arduino_nano

Commit message: Added C1 capacitor, changed jumper to solder joint, added own pogo pins adapter.
Parts:
- removed J1: Conn_01x03, Connector_PinHeader_2.54mm:PinHeader_1x03_P2.54mm_Vertical
- added C1: C, Capacitor_SMD:C_0805_2012Metric_Pad1.18x1.45mm_HandSolder, F.Cu at (171.4, 87.4)
- added JP1: SolderJumper_2_Bridged, Jumper:SolderJumper-2_P1.3mm_Bridged_RoundedPad1.0x1.5mm, F.Cu at (174.0, 87.0)
- added JP2: SolderJumper_3_Bridged12, Jumper:SolderJumper-3_P1.3mm_Bridged12_RoundedPad1.0x1.5mm, F.Cu at (177.2, 87.2)
- added h1: MountingHole_2.7mm_M2.5, MountingHole:MountingHole_2.7mm_M2.5, F.Cu at (191.8, 74.3)
- added h2: MountingHole_2.7mm_M2.5, MountingHole:MountingHole_2.7mm_M2.5, F.Cu at (191.8, 88.3)
Routing:
- net GND: track 2.43 -> 128.4 mm, vias 6 -> 8
- net Net-(JP1-Pad2): track 0.00 -> 16.3 mm
- net Net-(J2-Pad4): track 42.2 -> 31.3 mm
- net +3V3: track 43.2 -> 47.1 mm
- net Net-(C1-Pad1): track 0.00 -> 2.77 mm
- net Net-(J2-Pad3): track 66.3 -> 64.2 mm, vias 1 -> 0
- net +5V: track 22.9 -> 21.1 mm
- net Net-(J2-Pad1): track 71.3 -> 70.0 mm
- net Net-(J2-Pad2): track 74.1 -> 73.2 mm
Other:
- board text added: "Arduino Nano as ISP v1.1, 2021-03 CC BY-SA A. Suter crox.net/pcb"
- board text added: "G"
- board text added: "MI"
- board text added: "MO"
- board text removed: "Arduino Nano as ISP v1.0, 2021-01 CC BY-SA A. Suter crox.net/pcb"
- board text removed: "GND"
- board text removed: "MISO"
- board text removed: "MOSI"
